File: sram.kicad_sch (KiCad schematic)
At the start: 7 parts, among them U10N24 6116, U10N28 '32 - '256, U10N32 '512, U10W24 6116, U10W28 '32 - '256, U10W32 '512, X99 WE/A11

Commit message: updates
Parts:
- X21: renamed from X99; value WE/A11 -> A11/WE; footprint Jumper:SolderJumper-3_P1.3mm_Bridged12_RoundedPad1.0x1.5mm_NumberLabels -> MyPassives:SolderJumper-3_Pie_Bridged12
- renumbered U10N24 to U10
Changed lines of the file:
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@@
   (symbol (lib_name "6116_1") (lib_id "MyRam:6116") (at 50.8 78.74 0) (unit 1)
     (in_bom yes) (on_board yes) (fields_autoplaced)
-    (property "Reference" "U10N24" (id 0) (at 50.8 43.18 0))
+    (property "Reference" "U10" (id 0) (at 50.8 43.18 0))
     (property "Value" "6116" (id 1) (at 50.8 45.72 0))
     (property "Footprint" "MyPackages:DIP-24_W7.62mm" (id 2) (at 24.13 92.71 0)
@@
   (symbol (lib_id "Jumper:SolderJumper_3_Bridged12") (at 25.4 83.82 90) (unit 1)
     (in_bom yes) (on_board yes) (fields_autoplaced)
-    (property "Reference" "X99" (id 0) (at 22.86 82.5499 90)
+    (property "Reference" "X21" (id 0) (at 22.86 82.5499 90)
       (effects (font (size 1.27 1.27)) (justify left))
     )
-    (property "Value" "WE/A11" (id 1) (at 22.86 85.0899 90)
+    (property "Value" "A11/WE" (id 1) (at 22.86 85.0899 90)
       (effects (font (size 1.27 1.27)) (justify left))
     )
-    (property "Footprint" "Jumper:SolderJumper-3_P1.3mm_Bridged12_RoundedPad1.0x1.5mm_NumberLabels" (id 2) (at 25.4 83.82 0)
+    (property "Footprint" "MyPassives:SolderJumper-3_Pie_Bridged12" (id 2) (at 25.4 83.82 0)
       (effects (font (size 1.27 1.27)) hide)
     )
