File: 80ColumnCard.kicad_sch (KiCad schematic)
At the start: 41 parts, among them J1 Apple II Expansion Bus, J2 VIDEO & LIGHT PEN, Q1 2N3904, U1 74LS86, U10 CY7C128, U10B1 CY7C199, U14 74LS157, U15 74LS157, U16 74LS157, U18 74LS273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

Commit message: allow bigger RAM and ROM chips
Parts:
- removed U10: CY7C128, MyPackages:DIP-24_W7.62mm, symbol MyRam:6116
- removed U10B1: CY7C199, MyPackages:DIP-28_W7.62mm, symbol Memory_RAM:CY7C199
- removed U20: 2732, MyPackages:DIP-24_W15.24mm, symbol MyEprom:2732
- removed X1: U10: CY7C128* vs CY7C199, Jumper:SolderJumper-3_P1.3mm_Bridged12_RoundedPad1.0x1.5mm_NumberLabels, symbol Jumper:SolderJumper_3_Bridged12
- U3: value 2758 -> 2758/16/32
Connections:
- net SRAM/RAM_R/~{W}: now reaches U9.12 (O0)
- net RAMA0 renamed SRAM/RAMA0
- net RAMA1 renamed SRAM/RAMA1
- net RAMA10 renamed SRAM/RAMA10
- net RAMA11 renamed SRAM/RAMA11
- net RAMA2 renamed SRAM/RAMA2
- net RAMA3 renamed SRAM/RAMA3
- net RAMA4 renamed SRAM/RAMA4
- net RAMA5 renamed SRAM/RAMA5
- net RAMA6 renamed SRAM/RAMA6
- net RAMA7 renamed SRAM/RAMA7
- net RAMA8 renamed SRAM/RAMA8
- net RAMA9 renamed SRAM/RAMA9
- net RAMAB renamed RAM_~{A}/B
Other:
- added sheet Character ROM (char_rom.kicad_sch)
- added sheet SRAM (sram.kicad_sch)

Commit message: updates
Parts:
- removed U3: 2758/16/32, MyPackages:DIP-24_W15.24mm, symbol ambassador:2758
Connections:
- net Firmware/A9: now reaches U6.3
- net Firmware/~{OE}: now reaches U2.13
Other:
- added sheet Firmware (firmware.kicad_sch)
