File: hardware/80ColumnCard/80ColumnCard.kicad_pcb (KiCad board)
At the start: 2 copper layers, 155.2 x 78.6 mm, 55 parts, among them J1 Apple II Expansion Bus, J2 VIDEO & LIGHT PEN, Q1 2N3904, U1 74LS86, U10 6116, U10N28 '32 - '256, U10N32 '512, U10W24 6116, U10W28 '32 - '256, U10W32 '512, U14 74LS157, U15 74LS157, U16 74LS157, U18 74LS273, U19 MC6845, U2 74LS02, U20 2732, U20W28 '64 - '512, U21 74LS166, U22 74LS175, U23 74LS161, U3 2758/'16/'32, U3W28 '64 - '512, U4 74LS04, U5 74LS245, U6 74LS00, U7 4013, U8 4013, U9 74LS139, X21 A11/WE, X6 CHAR INV, X7 SCREEN INV, Y1 17.430 MHZ

Commit message: fiddling
Parts:
- added R3: 10K, MyPassives:R_Axial_DIN0207_L6.3mm_D1.6mm_P10.16mm_Horizontal, F.Cu at (156.0, 110.5)
- added R4: 10K, MyPassives:R_Axial_DIN0207_L6.3mm_D1.6mm_P10.16mm_Horizontal, F.Cu at (163.8, 110.5)
- JP1: value A10 -> A11; footprint Connector_PinHeader_2.54mm:PinHeader_1x03_P2.54mm_Vertical -> Connector_PinHeader_2.54mm:PinHeader_1x02_P2.54mm_Vertical
- JP2: value A11 -> A10; footprint Connector_PinHeader_2.54mm:PinHeader_1x03_P2.54mm_Vertical -> Connector_PinHeader_2.54mm:PinHeader_1x02_P2.54mm_Vertical
- JP7, JP8: value Jumper_2_Open -> Jumper_3_Bridged12; footprint Connector_PinHeader_2.54mm:PinHeader_1x02_P2.54mm_Vertical -> MyPassives:SolderJumper-3_Pie_Bridged12
- moved JP1 29.2 mm to (186.7, 100.3), turned to 90 degrees
- moved JP2 25.7 mm to (186.7, 105.4), turned to 90 degrees
- moved JP7 4.06 mm to (160.0, 115.3), turned to 90 degrees
- moved JP8 3.35 mm to (160.0, 108.4)
Connections:
- JP1 pad 1: GND -> /Firmware/A11
- JP1 pad 2: /Firmware/A10 -> +5V
- JP2 pad 1: GND -> /Firmware/A10
- JP2 pad 2: /Firmware/A11 -> +5V
- JP7 pad 1: +12V -> GND
Routing:
- net /Firmware/A11: track 31.2 -> 38.6 mm, vias 2 -> 3
- net GND: track 842.6 -> 848.6 mm
- net /Firmware/~{OE}: track 29.9 -> 25.1 mm
- net -5V: track 196.7 -> 201.1 mm, vias 3 -> 4
- net +12V: track 144.9 -> 149.1 mm, vias 0 -> 1
- net /A0: track 109.9 -> 113.4 mm
- net /R/~{W}: track 132.1 -> 134.4 mm
- net /A1: track 122.8 -> 120.5 mm
- net +5V: track 825.0 -> 826.4 mm, vias 4 -> 5
- net /Q3: track 65.9 -> 67.1 mm
- net /A10: track 99.2 -> 100.2 mm
- net /Firmware/A10: track 30.5 -> 31.5 mm
- net /A2: track 136.3 -> 137.0 mm
- net /D1: track 80.4 -> 81.1 mm
Other:
- board text added: "github.com/btb/80ColumnCard"
- board text removed: "FW SEL"
- board text removed: "btb"

Commit message: revert fiddling
Parts:
- removed JP1: A11, Connector_PinHeader_2.54mm:PinHeader_1x02_P2.54mm_Vertical
- removed JP2: A10, Connector_PinHeader_2.54mm:PinHeader_1x02_P2.54mm_Vertical
- removed JP3: A12, Connector_PinHeader_2.54mm:PinHeader_1x03_P2.54mm_Vertical
- removed JP4: A13, Connector_PinHeader_2.54mm:PinHeader_1x03_P2.54mm_Vertical
- removed JP5: A14, Connector_PinHeader_2.54mm:PinHeader_1x03_P2.54mm_Vertical
- removed JP6: A15, Connector_PinHeader_2.54mm:PinHeader_1x03_P2.54mm_Vertical
- removed JP7, JP8: Jumper_3_Bridged12, MyPassives:SolderJumper-3_Pie_Bridged12
- removed R3, R4: 10K, MyPassives:R_Axial_DIN0207_L6.3mm_D1.6mm_P10.16mm_Horizontal
- added U20C1: '010 - '080, Package_DIP:DIP-32_W15.24mm, F.Cu at (156.2, 72.4)
- C1, C4: footprint Capacitor_THT:CP_Radial_Tantal_D4.5mm_P5.00mm -> MyPassives:CP_Radial_Tantal_D4.5mm_P6.35mm
- C2, C3, C5: footprint Capacitor_THT:C_Disc_D4.3mm_W1.9mm_P5.00mm -> MyPassives:C_Axial_L2.6mm_D1.8mm_P6.35mm_Horizontal
- CR1: footprint Diode_THT:D_DO-35_SOD27_P7.62mm_Horizontal -> Diode_THT:D_DO-35_SOD27_P10.16mm_Horizontal
- moved C1 16.2 mm to (190.5, 106.7), turned to 90 degrees
- moved U16 5.08 mm to (149.9, 100.3)
- moved U20 3.81 mm to (166.4, 72.4)
- moved U20B1 3.81 mm to (161.3, 72.4)
- moved U15 2.54 mm to (134.6, 100.3)
- moved C2 1.27 mm to (212.7, 90.2)
- renumbered U20W28 to U20B1
Connections:
- net /DEVICE_SELECT renamed /DEV
- net /~{DEVICE_SELECT} renamed /~{DEV}
- U16 pad 13: /B11 -> GND
- U19 pad 15: /B11 -> unconnected-(U19-Pad15)
- U20 pad 24: /Character ROM/ROMA9 -> +5V
- U20B1 pad 1: /Character ROM/ROMA11 -> +5V
- U20B1 pad 2: /Character ROM/ROMA8 -> +5V
- U20B1 pad 26: /Character ROM/ROMA9 -> +5V
- U20B1 pad 27: /Character ROM/ROMA10 -> +5V
- U3 pad 19: /Firmware/A10 -> GND
- U3 pad 21: /Firmware/A11 -> +5V
- U3W28 pad 21: /Firmware/A10 -> GND
- U3W28 pad 23: /Firmware/A11 -> +5V
Routing:
- net /Firmware/A11: track 38.6 -> 0.00 mm, vias 3 -> 0
- net GND: track 848.6 -> 816.5 mm
- net /Firmware/A10: track 31.5 -> 0.00 mm
- net /Character ROM/ROMA8: track 24.0 -> 0.00 mm
- net /Character ROM/ROMA10: track 22.5 -> 0.00 mm
- net /D6: track 101.0 -> 80.1 mm
- net /Character ROM/ROMA9: track 20.3 -> 0.00 mm
- net -5V: track 201.1 -> 215.8 mm, vias 4 -> 3
- net /B11: track 13.4 -> 0.00 mm
- net /RAM_~{A}/B: track 218.8 -> 206.6 mm
- net Net-(Q1-Pad2): track 152.0 -> 140.4 mm
- net /RA0: track 81.1 -> 69.5 mm
- net /Character ROM/ROMA11: track 11.5 -> 0.00 mm
- net /RA1: track 75.5 -> 65.2 mm
- net Net-(U18-Pad11): track 199.0 -> 189.8 mm
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Other:
- board text added: "btb"
- board text removed: "C1: only needed for light pen or 2708"
- board text removed: "C4: optional"
- board text removed: "CHAR SEL"
- board text removed: "HI"
- board text removed: "LO"
- board text removed: "github.com/btb/80ColumnCard"

Commit message: Kicad 7, miscellaneous tweaks
Parts:
- removed U20C1: '010 - '080, Package_DIP:DIP-32_W15.24mm
Connections:
- net /DEV renamed /DEVSEL
- net /~{DEV} renamed /~{DEVSEL}
- net /~{IO_SELECT} renamed /~{IOSEL}
- net /~{IO_STROBE} renamed /~{IOSTRB}
- net Net-(CR1-Pad1) renamed /CA00
- net Net-(U1-Pad6) renamed /IOSEL
- net Net-(U2-Pad5) renamed /~{FF}
- net Net-(U21-Pad7) renamed /CLK
- net Net-(U7-Pad3) renamed /CE00
Routing:
- net +5V: track 834.8 -> 806.5 mm
Other:
- board text added: "github.com/btb/80ColumnCard"
- board text added: "rev ${REVISION}"
- board text removed: "btb"
