File: hardware/80ColumnCard/80ColumnCard.kicad_sch (KiCad schematic)
At the start: 36 parts, among them J1 Apple II Expansion Bus, J2 VIDEO & LIGHT PEN, Q1 2N3904, U1 74LS86, U14 74LS157, U15 74LS157, U16 74LS157, U18 74LS273, U19 MC6845, U2 74LS02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

Commit message: revert fiddling
Parts:
- removed C5: .1uF, Capacitor_THT:C_Disc_D4.3mm_W1.9mm_P5.00mm, symbol Device:C_Polarized
- added C5: .1uF, MyPassives:C_Axial_L2.6mm_D1.8mm_P6.35mm_Horizontal, symbol Device:C
- C1, C4: footprint Capacitor_THT:CP_Radial_Tantal_D4.5mm_P5.00mm -> MyPassives:CP_Radial_Tantal_D4.5mm_P6.35mm
- C2, C3: footprint Capacitor_THT:C_Disc_D4.3mm_W1.9mm_P5.00mm -> MyPassives:C_Axial_L2.6mm_D1.8mm_P6.35mm_Horizontal
- CR1: footprint Diode_THT:D_DO-35_SOD27_P7.62mm_Horizontal -> Diode_THT:D_DO-35_SOD27_P10.16mm_Horizontal
Connections:
- net +5V: now also C5.1
- net GND: now also U16.13 (I1d), C5.2
- net B11: no longer names the net of U19.15 (MA11)
- net B11: no longer U16.13 (I1d)
- net DEVICE_SELECT renamed DEV
- net ~{DEVICE_SELECT} renamed ~{DEV}
- no-connect marks 21 -> 36
Other:
- note removed: "Start at 4 or 5 and count up to 12 to draw either 8 or 9 pixels"
- title: (none) -> 80 Column Display
- moved on the sheet: C3, J1, R1, R2, R8, U1D, U1E, U21, U22, U23, U2E, U4C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

Commit message: Kicad 7, miscellaneous tweaks
Connections:
- net ~{FF}: now reaches U2.5, U7.2 (~{Q})
- net CA00: now reaches CR1.1 (K), U4.13, U9.5 (O1)
- net CE00: now reaches U7.3 (C), U9.7 (O3)
- net IOSEL: now reaches U1.6, U2.12, U7.6 (S)
- net CLK: now reaches U21.7 (Clk), U23.2 (CP), U4.10
- net DEV renamed DEVSEL
- net ~{DEV} renamed ~{DEVSEL}
- net ~{IO_SELECT} renamed ~{IOSEL}
- net ~{IO_STROBE} renamed ~{IOSTRB}
Other:
- note added: "C800 CA00 CC00 CE00"
- note added: "FW_A9 = A9 OR IOSEL FW_OE = (~{A10} AND IOSTRB AND FF) OR IOSEL"
- note added: "n = slot m = slot + 8 ~{DEVSEL} ~= C0m0 - C0mF ~{IOSEL} ~= Cn00 - CnFF ~{IOSTRB} ~= C800 - CFFF"
- moved on the sheet: C1, C2, C3, C4, C5, CR1, J2, Q1, R1, R10, R11, R12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
