File: hardware/80ColumnCard/firmware.kicad_sch (KiCad schematic)
At the start: 2 parts, among them U3 2758/'16/'32, U3W28 '64 - '512

Commit message: connect CRTC A11 to SRAM multiplexer. add jumpers for selectable firmware
Parts:
- added JP1: A10, Connector_PinHeader_2.54mm:PinHeader_1x03_P2.54mm_Vertical, symbol Jumper:Jumper_3_Open
- added JP2: A11, Connector_PinHeader_2.54mm:PinHeader_1x03_P2.54mm_Vertical, symbol Jumper:Jumper_3_Open
Connections:
- net +5V: now also JP1.3 (B), JP2.3 (B); no longer U3.21 (VPP), U3W28.23 (A11)
- net GND: now also JP1.1 (A), JP2.1 (A); no longer U3.19 (A10), U3W28.21 (A10)
- new net: JP1.2 (C), U3.19 (ARef/A10), U3W28.21 (A10)
- new net: JP2.2 (C), U3.21 (VPP/A11), U3W28.23 (A11)
Changed lines of the file:
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@@
   (junction (at 78.74 40.64) (diameter 0) (color 0 0 0 0)
   )
+  (junction (at 63.5 68.58) (diameter 0) (color 0 0 0 0)
+  )
   (junction (at 137.16 52.07) (diameter 0) (color 0 0 0 0)
   )
-  (junction (at 63.5 68.58) (diameter 0) (color 0 0 0 0)
+  (junction (at 30.48 57.15) (diameter 0) (color 0 0 0 0)
   )
   (junction (at 78.74 63.5) (diameter 0) (color 0 0 0 0)
@@
   (junction (at 137.16 54.61) (diameter 0) (color 0 0 0 0)
   )
+  (junction (at 30.48 74.93) (diameter 0) (color 0 0 0 0)
+  )
   (junction (at 78.74 38.1) (diameter 0) (color 0 0 0 0)
   )
@@
   (junction (at 137.16 46.99) (diameter 0) (color 0 0 0 0)
   )
-  (junction (at 63.5 66.04) (diameter 0) (color 0 0 0 0)
-  )
   (junction (at 137.16 41.91) (diameter 0) (color 0 0 0 0)
   )
@@
     (stroke (width 0) (type default) (color 0 0 0 0))
   )
-  (wire (pts (xy 63.5 71.12) (xy 63.5 68.58))
+  (wire (pts (xy 40.64 59.69) (xy 40.64 57.15))
     (stroke (width 0) (type default) (color 0 0 0 0))
   )
@@
     (stroke (width 0) (type default) (color 0 0 0 0))
   )
+  (wire (pts (xy 63.5 68.58) (xy 116.84 68.58))
+    (stroke (width 0) (type default) (color 0 0 0 0))
+  )
   (wire (pts (xy 152.4 44.45) (xy 137.16 44.45))
     (stroke (width 0) (type default) (color 0 0 0 0))
@@
     (stroke (width 0) (type default) (color 0 0 0 0))
   )
-  (wire (pts (xy 63.5 68.58) (xy 116.84 68.58))
+  (wire (pts (xy 40.64 57.15) (xy 30.48 57.15))
     (stroke (width 0) (type default) (color 0 0 0 0))
   )
@@
     (stroke (width 0) (type default) (color 0 0 0 0))
   )
+  (wire (pts (xy 63.5 68.58) (xy 63.5 71.12))
+    (stroke (width 0) (type default) (color 0 0 0 0))
+  )
   (wire (pts (xy 152.4 54.61) (xy 137.16 54.61))
     (stroke (width 0) (type default) (color 0 0 0 0))
   )
+  (wire (pts (xy 25.4 57.15) (xy 30.48 57.15))
+    (stroke (width 0) (type default) (color 0 0 0 0))
+  )
   (wire (pts (xy 78.74 71.12) (xy 116.84 71.12))
     (stroke (width 0) (type default) (color 0 0 0 0))
   )
+  (wire (pts (xy 25.4 74.93) (xy 30.48 74.93))
+    (stroke (width 0) (type default) (color 0 0 0 0))
+  )
   (wire (pts (xy 152.4 52.07) (xy 137.16 52.07))
     (stroke (width 0) (type default) (color 0 0 0 0))
@@
     (stroke (width 0) (type default) (color 0 0 0 0))
   )
+  (wire (pts (xy 30.48 74.93) (xy 40.64 74.93))
+    (stroke (width 0) (type default) (color 0 0 0 0))
+  )
   (wire (pts (xy 116.84 73.66) (xy 63.5 73.66))
     (stroke (width 0) (type default) (color 0 0 0 0))
   )
+  (wire (pts (xy 40.64 74.93) (xy 40.64 72.39))
+    (stroke (width 0) (type default) (color 0 0 0 0))
+  )
   (wire (pts (xy 88.9 86.36) (xy 127 86.36))
     (stroke (width 0) (type default) (color 0 0 0 0))
@@
     (stroke (width 0) (type default) (color 0 0 0 0))
   )
-  (wire (pts (xy 63.5 63.5) (xy 78.74 63.5))
+  (wire (pts (xy 34.29 63.5) (xy 78.74 63.5))
     (stroke (width 0) (type default) (color 0 0 0 0))
   )
@@
     (stroke (width 0) (type default) (color 0 0 0 0))
   )
-  (wire (pts (xy 63.5 66.04) (xy 78.74 66.04))
-    (stroke (width 0) (type default) (color 0 0 0 0))
-  )
-  (wire (pts (xy 63.5 68.58) (xy 63.5 66.04))
+  (wire (pts (xy 30.48 69.85) (xy 30.48 74.93))
+    (stroke (width 0) (type default) (color 0 0 0 0))
+  )
+  (wire (pts (xy 44.45 66.04) (xy 78.74 66.04))
     (stroke (width 0) (type default) (color 0 0 0 0))
   )
@@
   (hierarchical_label "A5" (shape input) (at 63.5 50.8 180)
     (effects (font (size 1.27 1.27)) (justify right))
+  )
+  (symbol (lib_id "power:+5V") (at 25.4 57.15 90) (unit 1)
+    (in_bom yes) (on_board yes) (fields_autoplaced)
+    (property "Reference" "#PWR0109" (id 0) (at 29.21 57.15 0)
+      (effects (font (size 1.27 1.27)) hide)
+    )
+    (property "Value" "+5V" (id 1) (at 24.13 53.34 90))
+    (property "Footprint" "" (id 2) (at 25.4 57.15 0)
+      (effects (font (size 1.27 1.27)) hide)
+    )
+    (property "Datasheet" "" (id 3) (at 25.4 57.15 0)
+      (effects (font (size 1.27 1.27)) hide)
+    )
+    (pin "1")
   )
   (symbol (lib_id "Memory_EPROM:2764") (at 127 58.42 0) (unit 1)
@@
     (pin "9")
   )
+  (symbol (lib_id "Jumper:Jumper_3_Open") (at 30.48 63.5 90) (unit 1)
+    (in_bom yes) (on_board yes) (fields_autoplaced)
+    (property "Reference" "JP1" (id 0) (at 27.94 62.2299 90)
+      (effects (font (size 1.27 1.27)) (justify left))
+    )
+    (property "Value" "A10" (id 1) (at 27.94 64.7699 90)
+      (effects (font (size 1.27 1.27)) (justify left))
+    )
+    (property "Footprint" "Connector_PinHeader_2.54mm:PinHeader_1x03_P2.54mm_Vertical" (id 2) (at 30.48 63.5 0)
+      (effects (font (size 1.27 1.27)) hide)
+    )
+    (property "Datasheet" "~" (id 3) (at 30.48 63.5 0)
+      (effects (font (size 1.27 1.27)) hide)
+    )
+    (pin "1")
+    (pin "2")
+    (pin "3")
+  )
   (symbol (lib_id "power:GND") (at 63.5 86.36 0) (unit 1)
     (in_bom yes) (on_board yes) (fields_autoplaced)
@@
     (pin "9")
   )
-  (symbol (lib_id "power:+5V") (at 63.5 66.04 90) (unit 1)
-    (in_bom yes) (on_board yes) (fields_autoplaced)
-    (property "Reference" "#PWR0107" (id 0) (at 67.31 66.04 0)
-      (effects (font (size 1.27 1.27)) hide)
-    )
-    (property "Value" "+5V" (id 1) (at 59.69 66.0399 90)
-      (effects (font (size 1.27 1.27)) (justify left))
-    )
-    (property "Footprint" "" (id 2) (at 63.5 66.04 0)
-      (effects (font (size 1.27 1.27)) hide)
-    )
-    (property "Datasheet" "" (id 3) (at 63.5 66.04 0)
-      (effects (font (size 1.27 1.27)) hide)
-    )
-    (pin "1")
-  )
-  (symbol (lib_id "power:GND") (at 63.5 63.5 270) (unit 1)
-    (in_bom yes) (on_board yes) (fields_autoplaced)
-    (property "Reference" "#PWR0108" (id 0) (at 57.15 63.5 0)
-      (effects (font (size 1.27 1.27)) hide)
-    )
-    (property "Value" "GND" (id 1) (at 59.69 63.4999 90)
+  (symbol (lib_id "power:+5V") (at 63.5 68.58 90) (unit 1)
+    (in_bom yes) (on_board yes) (fields_autoplaced)
+    (property "Reference" "#PWR0107" (id 0) (at 67.31 68.58 0)
+      (effects (font (size 1.27 1.27)) hide)
+    )
+    (property "Value" "+5V" (id 1) (at 59.69 68.5799 90)
+      (effects (font (size 1.27 1.27)) (justify left))
+    )
+    (property "Footprint" "" (id 2) (at 63.5 68.58 0)
+      (effects (font (size 1.27 1.27)) hide)
+    )
+    (property "Datasheet" "" (id 3) (at 63.5 68.58 0)
+      (effects (font (size 1.27 1.27)) hide)
+    )
+    (pin "1")
+  )
+  (symbol (lib_id "Jumper:Jumper_3_Open") (at 40.64 66.04 90) (unit 1)
+    (in_bom yes) (on_board yes) (fields_autoplaced)
+    (property "Reference" "JP2" (id 0) (at 38.1 64.7699 90)
+      (effects (font (size 1.27 1.27)) (justify left))
+    )
+    (property "Value" "A11" (id 1) (at 38.1 67.3099 90)
+      (effects (font (size 1.27 1.27)) (justify left))
+    )
+    (property "Footprint" "Connector_PinHeader_2.54mm:PinHeader_1x03_P2.54mm_Vertical" (id 2) (at 40.64 66.04 0)
+      (effects (font (size 1.27 1.27)) hide)
+    )
+    (property "Datasheet" "~" (id 3) (at 40.64 66.04 0)
+      (effects (font (size 1.27 1.27)) hide)
+    )
+    (pin "1")
+    (pin "2")
+    (pin "3")
+  )
+  (symbol (lib_id "power:GND") (at 25.4 74.93 270) (unit 1)
+    (in_bom yes) (on_board yes) (fields_autoplaced)
+    (property "Reference" "#PWR0108" (id 0) (at 19.05 74.93 0)
+      (effects (font (size 1.27 1.27)) hide)
+    )
+    (property "Value" "GND" (id 1) (at 21.59 74.9299 90)
       (effects (font (size 1.27 1.27)) (justify right))
     )
-    (property "Footprint" "" (id 2) (at 63.5 63.5 0)
-      (effects (font (size 1.27 1.27)) hide)
-    )
-    (property "Datasheet" "" (id 3) (at 63.5 63.5 0)
-      (effects (font (size 1.27 1.27)) hide)
-    )
+    (property "Footprint" "" (id 2) (at 25.4 74.93 0)
+      (effects (font (size 1.27 1.27)) hide)
+    )
+    (property "Datasheet" "" (id 3) (at 25.4 74.93 0)
+      (effects (font (size 1.27 1.27)) hide)
+    )

Commit message: clean up, add jumpers for fw/char selection
Parts:
- added JP7, JP8: Jumper_2_Open, Connector_PinHeader_2.54mm:PinHeader_1x02_P2.54mm_Vertical, symbol Jumper:Jumper_2_Open
Connections:
- net A10: now reaches JP1.2 (C), U3.19 (ARef/A10), U3W28.21 (A10)
- net A10: now also JP7.2 (B)
- net A11: now reaches JP2.2 (C), U3.21 (VPP/A11), U3W28.23 (A11)
- net A11: now also JP8.2 (B)
- new net +12V: JP7.1 (A)
- new net -5V: JP8.1 (A)
Other:
- note added: "2708: JP1 +12V, JP2 -5V 2758A: JP1 LOW JP2 HIGH 2758B: JP1 HIGH JP2 HIGH 2716: JP2 HIGH"
- note added: "EPROMs larger than 2732 can be used for convenience, but only the top 4KB is addressable."
- moved on the sheet: JP1, JP2

Commit message: fiddling
Parts:
- removed JP1: A10, Connector_PinHeader_2.54mm:PinHeader_1x03_P2.54mm_Vertical, symbol Jumper:Jumper_3_Open
- removed JP2: A11, Connector_PinHeader_2.54mm:PinHeader_1x03_P2.54mm_Vertical, symbol Jumper:Jumper_3_Open
- removed JP7, JP8: Jumper_2_Open, Connector_PinHeader_2.54mm:PinHeader_1x02_P2.54mm_Vertical, symbol Jumper:Jumper_2_Open
- added JP1: A11, Connector_PinHeader_2.54mm:PinHeader_1x02_P2.54mm_Vertical, symbol Jumper:Jumper_2_Open
- added JP2: A10, Connector_PinHeader_2.54mm:PinHeader_1x02_P2.54mm_Vertical, symbol Jumper:Jumper_2_Open
- added JP7, JP8: Jumper_3_Bridged12, MyPassives:SolderJumper-3_Pie_Bridged12, symbol Jumper:Jumper_3_Bridged12
- added R3, R4: 10K, MyPassives:R_Axial_DIN0207_L6.3mm_D1.6mm_P10.16mm_Horizontal, symbol Device:R
Connections:
- net +12V: now also JP7.3 (B)
- net +5V: now also JP1.2 (B), JP2.2 (B), JP8.3 (B)
- net -5V: now also JP8.1 (A)
- net A10: now also JP2.1 (A), JP7.2 (C), R4.1
- net A11: now also JP1.1 (A), JP8.2 (C), R3.1
- net GND: now also JP7.1 (A), R3.2, R4.2
Other:
- note added: "2708: Cut JP9, join JP8, cut JP10, join JP7, populate C1 2758A: JP1 LOW JP2 HIGH 2758B: JP1 HIGH JP2 HIGH 2716: JP2 HIGH"
- note removed: "2708: JP1 +12V, JP2 -5V 2758A: JP1 LOW JP2 HIGH 2758B: JP1 HIGH JP2 HIGH 2716: JP2 HIGH"

Commit message: revert fiddling
Parts:
- removed JP1: A11, Connector_PinHeader_2.54mm:PinHeader_1x02_P2.54mm_Vertical, symbol Jumper:Jumper_2_Open
- removed JP2: A10, Connector_PinHeader_2.54mm:PinHeader_1x02_P2.54mm_Vertical, symbol Jumper:Jumper_2_Open
- removed JP7, JP8: Jumper_3_Bridged12, MyPassives:SolderJumper-3_Pie_Bridged12, symbol Jumper:Jumper_3_Bridged12
- removed R3, R4: 10K, MyPassives:R_Axial_DIN0207_L6.3mm_D1.6mm_P10.16mm_Horizontal, symbol Device:R
Connections:
- net A10 is gone; now on net GND: U3.19 (A10), U3W28.21 (A10)
- net A11 is gone; now on net +5V: U3.21 (VPP), U3W28.23 (A11)
Other:
- note removed: "2708: Cut JP9, join JP8, cut JP10, join JP7, populate C1 2758A: JP1 LOW JP2 HIGH 2758B: JP1 HIGH JP2 HIGH 2716: JP2 HIGH"
- note removed: "EPROMs larger than 2732 can be used for convenience, but only the top 4KB is addressable."
